File: Schematics/Arduino MEGA Tester/Arduino MEGA Tester Shield/Arduino Mega DRAM Tester Shield.brd (EAGLE design)
At the start: 120 x 80.2 mm, 40 parts, among them IC1 DPAN02E-05, IC2 SPAN02E12, U1 ARDUINO-MEGAFULL, X1 2524-, X2 2524-

Commit message: Moved a few I/O around. Added some pin mapping files. Adjusted OLED position.
Parts:
- moved S1 3.81 mm to (11.4, 20.3)
- moved S2 2.54 mm to (24.1, 20.3)
- moved U$1 2.54 mm to (24.1, 42.2)
- moved S3 1.90 mm to (37.5, 20.3)
Connections:
- removed net AB0: U1.A3, X1.5
- removed net AB1: U1.A4, X1.4
- removed net AB2: U1.A5, X1.3
- removed net CA2: R27.1, U1.16
- removed net CA2X: IC4.14, R27.2
- new net CA4: R25.1, U1.7
- new net CA4X: IC4.12, R25.2, X2.11
- net CA0: now also R27.1, U1.16; no longer R25.1, U1.14
- net CA0X: now also IC4.14, R27.2, X2.14; no longer IC4.12, R25.2
- net CA1: now also R28.1, U1.17; no longer R26.1, U1.15
- net CA1X: now also IC4.15, R28.2, X2.13; no longer IC4.13, R26.2
- net CA3: now also R26.1, U1.6; no longer R28.1, U1.17
- net CA3X: now also IC4.13, R26.2, X2.12; no longer IC4.15, R28.2
- net CB0: now also U1.10, X1.5; no longer U1.50, X2.14
- net CB1: now also U1.11, X1.4; no longer U1.51, X2.13
- net CB2: now also U1.12, X1.3; no longer U1.52, X2.12
- net CB3: now also U1.13, X1.2; no longer U1.53, X2.11
- net GND: no longer X1.2
Routing:
- net AB2: track 32.9 -> 0.00 mm
- net AB1: track 32.4 -> 0.00 mm
- net CA4X: track 0.00 -> 28.3 mm
- net CA4: track 0.00 -> 28.1 mm
- net CA3: track 4.80 -> 32.6 mm
- net CB3: track 23.3 -> 48.9 mm
- net CB2: track 23.6 -> 48.9 mm
- net AB0: track 23.0 -> 0.00 mm
- net CB1: track 22.8 -> 41.9 mm
- net CB0: track 23.2 -> 39.4 mm
- net CA3X: track 10.5 -> 22.6 mm
- net CA2X: track 11.8 -> 0.00 mm
- net SCL: track 6.03 -> 14.3 mm
- net CA1X: track 14.4 -> 22.7 mm
- net CA2: track 4.80 -> 0.00 mm
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