File: Schematics/Arduino MEGA Tester/Arduino MEGA Tester Shield/Arduino Mega DRAM Tester Shield.sch (EAGLE design)
At the start: 40 parts, among them IC1 DPAN02E-05, IC2 SPAN02E12, U1 ARDUINO-MEGAFULL, X1 2524-, X2 2524-

Commit message: Moved a few I/O around. Added some pin mapping files. Adjusted OLED position.
Connections:
- removed net AB0: U1.A3, X1-5.KL
- removed net AB1: U1.A4, X1-4.KL
- removed net AB2: U1.A5, X1-3.KL
- removed net CA2: R27.1, U1.16(TX2)
- removed net CA2X: IC4.IN13, R27.2
- new net CA4: R25.1, U1.7
- new net CA4X: IC4.IN11, R25.2, X2-11.KL
- net CA0: now also R27.1, U1.16(TX2); no longer R25.1, U1.14(TX3)
- net CA0X: now also IC4.IN13, R27.2, X2-14.KL; no longer IC4.IN11, R25.2
- net CA1: now also R28.1, U1.17(RX2); no longer R26.1, U1.15(RX3)
- net CA1X: now also IC4.IN14, R28.2, X2-13.KL; no longer IC4.IN12, R26.2
- net CA3: now also R26.1, U1.6; no longer R28.1, U1.17(RX2)
- net CA3X: now also IC4.IN12, R26.2, X2-12.KL; no longer IC4.IN14, R28.2
- net CB0: now also U1.10, X1-5.KL; no longer U1.50, X2-14.KL
- net CB1: now also U1.11, X1-4.KL; no longer U1.51, X2-13.KL
- net CB2: now also U1.12, X1-3.KL; no longer U1.52, X2-12.KL
- net CB3: now also U1.13, X1-2.KL; no longer U1.53, X2-11.KL
- net GND: no longer X1-2.KL
